Commit message: Changes in ur_common.xacro

File: urdf/inc/ur_common.xacro (robot description, xacro)
@@ -30,5 +30,5 @@
     </xacro:if>
     <xacro:unless value="${force_abs_paths}">
-      <xacro:property name="mesh" value="package://${visual_params['mesh']['package']}/${visual_params['mesh']['path']}" scope="parent"/>
+      <xacro:property name="mesh" value="file://$(find ${visual_params['mesh']['package']})/${visual_params['mesh']['path']}" scope="parent"/>
     </xacro:unless>
   </xacro:macro>
